Commit message: update for panda wrist cam

File: mani_skill/assets/robots/panda/panda_v3.urdf (robot description, URDF)
Before this commit: robot panda, 15 links, 14 joints
Links:
- link camera_link: geometry collision box size=0.02005 0.099 0.023; visual mesh filename=realsense2_description/meshes/d435.dae
Joints:
- joint camera_link_joint: origin xyz=0 0.02 0.0115 rpy=0 0 0 -> xyz=-0.03 0.0 0.05 rpy=0 0.436 0
